File: control_neumatica/control_neumatica.kicad_pcb (KiCad board)
At the start: 2 copper layers, 38.7 x 42.5 mm, 11 parts

Commit message: version v2
Parts:
- removed the   at (136.3, 57.5)
- removed the   at (136.3, 52.1)
- removed GND      12V: Screw_Terminal_01x02, Connector_Phoenix_MC_HighVoltage:PhoenixContact_MCV_1,5_2-G-5.08_1x02_P5.08mm_Vertical
- removed the SALIDAS                12V at (151.8, 42.8)
- removed the X              ENTRADAS at (125.0, 50.5)
- added  : Conn_01x03_Male, Connector_PinSocket_2.54mm:PinSocket_1x03_P2.54mm_Vertical, F.Cu at (136.3, 57.1)
- added  : Screw_Terminal_01x02, Conector_Eurobot:Conector_2p_5.08, F.Cu at (138.7, 41.7)
- added  : Conn_01x03_Male, Connector_PinSocket_2.54mm:PinSocket_1x03_P2.54mm_Vertical, F.Cu at (136.3, 50.8)
- added ?: , , F.Cu at (273.6, 129.9)
- added ? (x2): , , F.Cu at (138.4, 72.6)
- added ?: , , F.Cu at (141.1, 73.5)
- added ?: , , F.Cu at (139.2, 79.0)
- added ?: , , F.Cu at (139.6, 73.3)
- added SALIDAS                12V: Salida 12v, Conector_Eurobot:Conector_6p_5.08, F.Cu at (152.7, 55.9)
- added X              ENTRADAS: Entrada Digital, Conector_Eurobot:Conector_6p_5.08, F.Cu at (125.0, 63.2)
- S  D  G: renamed from S   D   G
- moved S  D  G 2.59 mm to (136.2, 76.2)
- moved   1.42 mm to (136.2, 69.8)
- moved   0.51 mm to (136.3, 63.5)
Routing:
- net O4: track 16.2 -> 19.3 mm
- net O5: track 16.2 -> 18.5 mm
- net O3: track 16.0 -> 17.9 mm
- net +12V: track 10.3 -> 12.1 mm
- net O1: track 15.7 -> 16.9 mm
- net O2: track 15.8 -> 17.0 mm
- net I5: track 17.5 -> 18.6 mm
- net I1: track 17.0 -> 18.1 mm
- net I2: track 17.1 -> 18.0 mm
- net I4: track 17.4 -> 18.0 mm
