File: potencia sin fusibles/potencia.kicad_pcb (KiCad board)
At the start: 2 copper layers, 82 x 115.3 mm, 18 parts

Commit message: v2
Routing:
- net 5.2: track 103.2 -> 143.4 mm, vias 0 -> 2
- net +BATT: track 174.2 -> 185.3 mm
- net GND: track 104.2 -> 93.8 mm
- net +15V: track 116.5 -> 110.0 mm, vias 0 -> 2
- net 5.1: track 42.6 -> 38.1 mm, vias 0 -> 2
- net 12.1: track 63.2 -> 59.2 mm, vias 0 -> 2
- net 12.2: track 187.5 -> 187.0 mm
Other:
- board text added: "SIN POSAVASOS V2"
- board text removed: "SIN POSAVASOS"

Commit message: version v2
Parts:
- removed 5V    5V    5V    GND    12V    12V: Screw_Terminal_01x06, Connector_Phoenix_MC_HighVoltage:PhoenixContact_MCV_1,5_6-G-5.08_1x06_P5.08mm_Vertical
- removed GND    5V    12V    GND: Screw_Terminal_01x04, Connector_Phoenix_MC_HighVoltage:PhoenixContact_MCV_1,5_4-G-5.08_1x04_P5.08mm_Vertical
- removed GND   GND   BAT   SETA: Screw_Terminal_01x04, Connector_Phoenix_MC_HighVoltage:PhoenixContact_MCV_1,5_4-G-5.08_1x04_P5.08mm_Vertical
- added Alimentación1: Screw_Terminal_01x04, Conector_Eurobot:Conector_4p_5.08, F.Cu at (125.7, 154.3)
- added Extra1: Screw_Terminal_01x04, Conector_Eurobot:Conector_4p_5.08, F.Cu at (181.6, 154.3)
- added R1: R, Resistor_THT:R_Axial_DIN0204_L3.6mm_D1.6mm_P5.08mm_Horizontal, F.Cu at (123.6, 141.5)
- added R2: R, Resistor_THT:R_Axial_DIN0204_L3.6mm_D1.6mm_P5.08mm_Horizontal, F.Cu at (162.0, 100.9)
- added R3: R, Resistor_THT:R_Axial_DIN0204_L3.6mm_D1.6mm_P5.08mm_Horizontal, F.Cu at (139.7, 66.4)
- added R4: R, Resistor_THT:R_Axial_DIN0204_L3.6mm_D1.6mm_P5.08mm_Horizontal, F.Cu at (180.7, 120.7)
- added R5: R, Resistor_THT:R_Axial_DIN0204_L3.6mm_D1.6mm_P5.08mm_Horizontal, F.Cu at (177.2, 62.0)
- added Salida1: Screw_Terminal_01x06, Conector_Eurobot:Conector_6p_5.08, F.Cu at (153.7, 154.3)
- H1, H2, H3, Regulador5.1, Regulador5.3: renamed from  
- Regulador5.2: renamed from   
- renumbered In- to NI12.1, In- to NI12.2, Out- to NO12.1, Out- to NO12.2, In+ to PI12.1, In+ to PI12.2, Out+ to PO12.1, Out+ to PO12.2
Routing:
- net Net-(Extra1-Pad3): track 0.00 -> 187.4 mm
- net 12.2: track 187.0 -> 9.03 mm
- net Net-(Extra1-Pad2): track 0.00 -> 134.4 mm, vias 0 -> 2
- net 5.2: track 143.4 -> 9.70 mm, vias 2 -> 0
- net Net-(F3-Pad2): track 0.00 -> 95.3 mm
- net GND: track 93.8 -> 0.72 mm
- net 5.3: track 101.2 -> 17.1 mm
- net Net-(F4-Pad2): track 0.00 -> 50.1 mm, vias 0 -> 1
- net 12.1: track 59.2 -> 16.4 mm, vias 2 -> 0
- net 5.1: track 38.1 -> 7.55 mm, vias 2 -> 0
- net Net-(F1-Pad2): track 0.00 -> 29.3 mm, vias 0 -> 1
- net +BATT: track 185.3 -> 159.5 mm, vias 0 -> 1
- net +15V: track 110.0 -> 120.4 mm
